File: ADR1399/ADR1399.kicad_sch (KiCad schematic)
At the start: 80 parts, among them J1 10V, J2 Conn_01x04_Male, J3 4V6, J4 7V, J5 Conn_01x02_Male, J6 Conn_01x02_Male, J7 Conn_01x01_Male, Q1 BC547, Q2 BC547, U1 OPA2182xD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

Commit message: Push the local work from Ryzen5600G PC part 1
Parts:
- removed J2: Conn_01x04_Male, Connector_PinHeader_2.54mm:PinHeader_1x04_P2.54mm_Vertical, symbol Connector:Conn_01x04_Male
- added J2: PT100, Connector_PinHeader_2.54mm:PinHeader_1x02_P2.54mm_Vertical, symbol Connector:Conn_01x02_Male
- CR1: value SZSMF4L12AT3G -> SZSMF4L12AT3G
- CR2: value SZSMF4L6.5AT3G -> SZSMF4L6.5AT3G
- CR3: value SZSMF4L8.5AT3G -> SZSMF4L8.5AT3G
- TH1: footprint Connector_PinHeader_2.54mm:PinHeader_2x02_P2.54mm_Vertical -> Connector_PinHeader_1.27mm:PinHeader_2x02_P1.27mm_Vertical
- TP1, TP2: value (none) -> ~
Connections:
- net at TH1.1, TH1.2: now also J2.2 (Pin_2)
- net at TH1.3, TH1.4: now also J2.1 (Pin_1)
