File: ADR1399New/_autosave-ADR1399.kicad_sch (KiCad schematic)
At the start: 79 parts, among them J1 10V, J2 PT100, J3 GNDF_SPARE, J4 7V, J5 Conn_01x02_Male, J6 Conn_01x02_Male, J7 Conn_01x01_Male, J8 Conn_01x02_Male, J9 Conn_01x02_Male, U1 OPA2182xD, U2 OPA2209xD, U3 OPA2182xD, U4 LM399, U5 LM7815_TO220, U6 LM7805_TO220, U8 LM7905_TO220

Commit message: Update KiCad project and add latest backups
Parts:
- removed C26: 100n, Capacitor_SMD:C_0805_2012Metric_Pad1.18x1.45mm_HandSolder, symbol Device:C
- removed C8: 2n2, Capacitor_SMD:C_0805_2012Metric_Pad1.18x1.45mm_HandSolder, symbol Device:C
- removed TH1: PT1000, Connector_PinHeader_1.27mm:PinHeader_2x02_P1.27mm_Vertical, symbol Device:Thermistor_PTC_4Wire
- added C30: 100n, Capacitor_SMD:C_0805_2012Metric_Pad1.18x1.45mm_HandSolder, symbol Device:C
- added H1, H2, H3, H4: 3mm, MountingHole:MountingHole_3.2mm_M3, symbol Mechanical:MountingHole
- added J4: Guards, Connector_PinHeader_2.54mm:PinHeader_2x02_P2.54mm_Vertical, symbol Connector:Conn_01x04_Pin
- added JP1: 3k3/5k, Jumper:SolderJumper-2_P1.3mm_Bridged2Bar_RoundedPad1.0x1.5mm, symbol Jumper:Jumper_2_Small_Bridged
- added JP2: 8k33/10k, Jumper:SolderJumper-2_P1.3mm_Bridged2Bar_RoundedPad1.0x1.5mm, symbol Jumper:Jumper_2_Small_Bridged
- added NT2: NetTie_2, NetTie:NetTie-2_SMD_Pad2.0mm, symbol Device:NetTie_2
- added NT3: NetTie_3, symbol Device:NetTie_3
- added Q1: BC817, Package_TO_SOT_SMD:SOT-23, symbol Transistor_BJT:BC817
- added R13, R6: 33, Resistor_SMD:R_0805_2012Metric_Pad1.20x1.40mm_HandSolder, symbol Device:R
- added TH1: PT1000, Connector_PinHeader_1.27mm:PinHeader_1x02_P1.27mm_Vertical, symbol Sensor_Temperature:PT1000
- C1: renamed from C14; value 2n -> 100n; footprint Capacitor_SMD:C_0805_2012Metric_Pad1.18x1.45mm_HandSolder -> Capacitor_SMD:C_1206_3216Metric_Pad1.33x1.80mm_HandSolder
- C10: renamed from C17; footprint Capacitor_THT:C_Rect_L7.2mm_W4.5mm_P5.00mm_FKS2_FKP2_MKS2_MKP2 -> Capacitor_THT:C_Rect_L7.2mm_W5.5mm_P5.00mm_FKS2_FKP2_MKS2_MKP2
- C11: renamed from C18; value 10n -> 1n
- C13: renamed from C20; value 22n -> 100n; footprint Capacitor_SMD:C_0805_2012Metric_Pad1.18x1.45mm_HandSolder -> Capacitor_SMD:C_1206_3216Metric_Pad1.33x1.80mm_HandSolder
- C15: renamed from C16; value 2n -> 100p; footprint Capacitor_SMD:C_0805_2012Metric_Pad1.18x1.45mm_HandSolder -> Capacitor_SMD:C_1206_3216Metric_Pad1.33x1.80mm_HandSolder
- C16: renamed from C34; footprint Capacitor_SMD:C_0805_2012Metric_Pad1.18x1.45mm_HandSolder -> Capacitor_SMD:C_1206_3216Metric_Pad1.33x1.80mm_HandSolder
- C17: renamed from C22; value C -> 100n; footprint Capacitor_SMD:C_1206_3216Metric -> Capacitor_SMD:C_1206_3216Metric_Pad1.33x1.80mm_HandSolder
- C19: renamed from C32; footprint Capacitor_SMD:C_1206_3216Metric -> Capacitor_Tantalum_SMD:CP_EIA-3528-12_Kemet-T_HandSolder
- C2: renamed from C35; footprint Capacitor_SMD:C_0805_2012Metric_Pad1.18x1.45mm_HandSolder -> Capacitor_SMD:C_1206_3216Metric_Pad1.33x1.80mm_HandSolder
- C25: renamed from C21; value C -> 100n; footprint Capacitor_SMD:C_1206_3216Metric -> Capacitor_SMD:C_1206_3216Metric_Pad1.33x1.80mm_HandSolder
- C27: renamed from C24; value 100.0 -> 220.0; footprint Capacitor_SMD:C_1206_3216Metric -> Capacitor_THT:CP_Radial_D10.0mm_P7.50mm
- C28: renamed from C25; footprint Capacitor_SMD:C_1206_3216Metric -> Capacitor_Tantalum_SMD:CP_EIA-3528-12_Kemet-T_HandSolder
- C3: renamed from C1; footprint Capacitor_THT:C_Rect_L7.2mm_W4.5mm_P5.00mm_FKS2_FKP2_MKS2_MKP2 -> Capacitor_THT:C_Rect_L7.2mm_W5.5mm_P5.00mm_FKS2_FKP2_MKS2_MKP2
- C4: renamed from C2; value 10n -> 1n
- C5: renamed from C3; footprint Capacitor_SMD:C_0805_2012Metric_Pad1.18x1.45mm_HandSolder -> Capacitor_SMD:C_1206_3216Metric_Pad1.33x1.80mm_HandSolder
- C6: renamed from C4; footprint Capacitor_SMD:C_0805_2012Metric_Pad1.18x1.45mm_HandSolder -> Capacitor_SMD:C_1206_3216Metric_Pad1.33x1.80mm_HandSolder
- C7: renamed from C5; footprint Capacitor_SMD:C_0805_2012Metric_Pad1.18x1.45mm_HandSolder -> Capacitor_SMD:C_1206_3216Metric_Pad1.33x1.80mm_HandSolder
- C8: renamed from C6; value 2n -> 100n; footprint Capacitor_SMD:C_0805_2012Metric_Pad1.18x1.45mm_HandSolder -> Capacitor_SMD:C_1206_3216Metric_Pad1.33x1.80mm_HandSolder
- C9: renamed from C7; value 10n -> 100n; footprint Capacitor_SMD:C_0805_2012Metric_Pad1.18x1.45mm_HandSolder -> Capacitor_SMD:C_1206_3216Metric_Pad1.33x1.80mm_HandSolder
- CR1: renamed from CR2; footprint TVS:ZDO_TPSMF4L5.0A_LTF -> TVS:ZDO_TPSMF4L5.0A_LTF-L
- CR2: renamed from CR1; footprint TVS:ZDO_TPSMF4L5.0A_LTF -> TVS:ZDO_TPSMF4L5.0A_LTF-L
- CR3: footprint TVS:ZDO_TPSMF4L5.0A_LTF -> TVS:ZDO_TPSMF4L5.0A_LTF-L
- J5: renamed from J4; footprint (none) -> Connector_PinHeader_2.54mm:PinHeader_1x04_P2.54mm_Vertical
- NT1: footprint (none) -> NetTie:NetTie-2_SMD_Pad2.0mm
- R1: renamed from R17; value 1k -> 220
- R11: renamed from R8; footprint Package_SO:SO-16_3.9x9.9mm_P1.27mm -> Package_SO:SOIC-16_3.9x9.9mm_P1.27mm
- R15: renamed from R16; value 470 -> 100
- R21: renamed from R14; value 1k -> 100
- R3: renamed from R2; value 2k7 -> 2k7/910; footprint Resistor_SMD:R_0805_2012Metric_Pad1.20x1.40mm_HandSolder -> Resistor_SMD:R_1206_3216Metric_Pad1.30x1.75mm_HandSolder
- R7: renamed from R4; value 1k -> 100
- renumbered C15 to C12, C19 to C14, C31 to C18, C30 to C21, C27 to C22, C28 to C23, C29 to C24, C23 to C26, C33 to C29, D3 to D1, D4 to D2, D1 to D3, D2 to D4, J3 to J1, J7 to J10, J1 to J2, J2 to J3, J8 to J6, J9 to J7, J5 to J8, J6 to J9, R7 to R10, R18 to R12, R15 to R14, R20 to R16, R21 to R17, R26 to R18, R22 to R19, R1 to R2, R19 to R20, R25 to R22, R27 to R23, R23 to R24, R28 to R4, R3 to R5, R29 to R8, R5 to R9, TP3 to TP1, U3 to U1, U1 to U3, U8 to U5, U5 to U6, U6 to U7
Connections:
- net +15V: now also NT2.1, Q1.3 (C); no longer C6.1, U4.3
- net 7V_force: no longer C14.2, R16.2, R19.2, TP2.1
- net GND: now also C21.2, C30.1, J4.1 (Pin_1), J4.2 (Pin_2)
- net GNDZ: now also R11.6, R11.7, R11.8, J4.3 (Pin_3), J4.4 (Pin_4); no longer R11.3
- net at R11.1: now also C9.2, R11.2, R11.3, R11.4, R11.5, U3.2 (-)
- net at R11.10, R11.11: now also R11.12, R11.13, JP2.1 (A); no longer R11.15
- net at R11.14: now also C5.1, C8.1, CR2.1, J2.2 (Pin_2), R10.1, R11.15, R7.2, U2.3 (+), JP1.2 (B); no longer R11.12
- net at R11.16: now also JP1.1 (A)
- net at R11.9: now also JP2.2 (B)
- net at C28.1, U1.8 (V+), U7.3 (VO): now also C30.2; no longer C21.2
- net at R3.2, U2.2 (-): now also Q1.2 (E); no longer U2.1
- net at C3.2, C4.1, R5.2: now also R6.1; no longer U3.3 (+)
- net at R15.1, U2.7: now also C14.2, R16.2, R19.2, TP2.1
- net at J3.1 (Pin_1): now also TH1.2
- net at J3.2 (Pin_2): now also TH1.1
- net at C10.2, C11.1, R12.2: now also R13.1; no longer U3.5 (+)
- new net: Q1.1 (B), U2.1
- new net: R13.2, U3.5 (+)
- new net: R6.2, U3.3 (+)
- new net +24V: C6.1, NT2.2, U4.3
- no-connect marks 4 -> 0
Other:
- moved on the sheet: C10, C11, C21, C3, C4, C7, CR3, R11, R12, R15, R3, R5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
