File: ADR1399New/ADR1399.kicad_pcb (KiCad board)
At the start: 4 copper layers, 108 x 55.5 mm, 76 parts, among them J1 10V, J2 PT100, J3 GNDF_SPARE, J5 Conn_01x02_Male, J6 Conn_01x02_Male, J7 Conn_01x01_Male, J8 Conn_01x02_Male, J9 Conn_01x02_Male, U1 OPA2182xD, U2 OPA2209xD, U3 OPA2182xD, U4 LM399, U5 LM7815_TO220, U6 LM7805_TO220, U8 LM7905_TO220

Commit message: Update KiCad project and add latest backups
Parts:
- removed the C26 at (108.4, 43.2)
- removed the C8 at (141.3, 52.0)
- added C30: 100n, Capacitor_SMD:C_0805_2012Metric_Pad1.18x1.45mm_HandSolder, F.Cu at (105.0, 62.0)
- added H1: 3mm, MountingHole:MountingHole_3.2mm_M3, F.Cu at (29.5, 24.5)
- added H2: 3mm, MountingHole:MountingHole_3.2mm_M3, F.Cu at (29.5, 71.0)
- added H3: 3mm, MountingHole:MountingHole_3.2mm_M3, F.Cu at (117.5, 24.0)
- added H4: 3mm, MountingHole:MountingHole_3.2mm_M3, F.Cu at (117.5, 72.0)
- added J4: Guards, Connector_PinHeader_2.54mm:PinHeader_2x02_P2.54mm_Vertical, F.Cu at (122.2, 30.2)
- added J5: 7V, Connector_PinHeader_2.54mm:PinHeader_1x04_P2.54mm_Vertical, F.Cu at (125.0, 56.5)
- added JP1: 3k3/5k, Jumper:SolderJumper-2_P1.3mm_Bridged2Bar_RoundedPad1.0x1.5mm, F.Cu at (83.0, 48.0)
- added JP2: 8k33/10k, Jumper:SolderJumper-2_P1.3mm_Bridged2Bar_RoundedPad1.0x1.5mm, F.Cu at (75.0, 48.0)
- added NT1: NetTie_2, NetTie:NetTie-2_SMD_Pad2.0mm, F.Cu at (60.0, 27.5)
- added NT2: NetTie_2, NetTie:NetTie-2_SMD_Pad2.0mm, F.Cu at (50.0, 49.0)
- added Q1: BC817, Package_TO_SOT_SMD:SOT-23, F.Cu at (73.0, 54.5)
- added R13: 33, Resistor_SMD:R_0805_2012Metric_Pad1.20x1.40mm_HandSolder, F.Cu at (85.5, 33.5)
- added R6: 33, Resistor_SMD:R_0805_2012Metric_Pad1.20x1.40mm_HandSolder, F.Cu at (85.5, 35.5)
- added TP1: GNDZ, TestPoint:TestPoint_Pad_1.5x1.5mm, F.Cu at (111.5, 33.5)
- C1: renamed from C14; value 2n -> 100n; footprint Capacitor_SMD:C_0805_2012Metric_Pad1.18x1.45mm_HandSolder -> Capacitor_SMD:C_1206_3216Metric_Pad1.33x1.80mm_HandSolder
- C10: renamed from C17; footprint Capacitor_THT:C_Rect_L7.2mm_W4.5mm_P5.00mm_FKS2_FKP2_MKS2_MKP2 -> Capacitor_THT:C_Rect_L7.2mm_W5.5mm_P5.00mm_FKS2_FKP2_MKS2_MKP2
- C11: renamed from C18; value 10n -> 1n
- C13: renamed from C20; value 22n -> 100n; footprint Capacitor_SMD:C_0805_2012Metric_Pad1.18x1.45mm_HandSolder -> Capacitor_SMD:C_1206_3216Metric_Pad1.33x1.80mm_HandSolder
- C15: renamed from C16; value 2n -> 100p; footprint Capacitor_SMD:C_0805_2012Metric_Pad1.18x1.45mm_HandSolder -> Capacitor_SMD:C_1206_3216Metric_Pad1.33x1.80mm_HandSolder
- C16: renamed from C34; footprint Capacitor_SMD:C_0805_2012Metric_Pad1.18x1.45mm_HandSolder -> Capacitor_SMD:C_1206_3216Metric_Pad1.33x1.80mm_HandSolder
- C17: renamed from C22; value C -> 100n; footprint Capacitor_SMD:C_1206_3216Metric -> Capacitor_SMD:C_1206_3216Metric_Pad1.33x1.80mm_HandSolder
- C19: renamed from C32; footprint Capacitor_SMD:C_1206_3216Metric -> Capacitor_Tantalum_SMD:CP_EIA-3528-12_Kemet-T_HandSolder
- C2: renamed from C35; footprint Capacitor_SMD:C_0805_2012Metric_Pad1.18x1.45mm_HandSolder -> Capacitor_SMD:C_1206_3216Metric_Pad1.33x1.80mm_HandSolder
- C25: renamed from C21; value C -> 100n; footprint Capacitor_SMD:C_1206_3216Metric -> Capacitor_SMD:C_1206_3216Metric_Pad1.33x1.80mm_HandSolder
- C27: renamed from C24; value 100.0 -> 220.0; footprint Capacitor_SMD:C_1206_3216Metric -> Capacitor_THT:CP_Radial_D10.0mm_P7.50mm
- C28: renamed from C25; footprint Capacitor_SMD:C_1206_3216Metric -> Capacitor_Tantalum_SMD:CP_EIA-3528-12_Kemet-T_HandSolder
- C3: renamed from C1; footprint Capacitor_THT:C_Rect_L7.2mm_W4.5mm_P5.00mm_FKS2_FKP2_MKS2_MKP2 -> Capacitor_THT:C_Rect_L7.2mm_W5.5mm_P5.00mm_FKS2_FKP2_MKS2_MKP2
- C4: renamed from C2; value 10n -> 1n
- C5: renamed from C3; footprint Capacitor_SMD:C_0805_2012Metric_Pad1.18x1.45mm_HandSolder -> Capacitor_SMD:C_1206_3216Metric_Pad1.33x1.80mm_HandSolder
- C6: renamed from C4; footprint Capacitor_SMD:C_0805_2012Metric_Pad1.18x1.45mm_HandSolder -> Capacitor_SMD:C_1206_3216Metric_Pad1.33x1.80mm_HandSolder; moved to B.Cu
- C7: renamed from C5; footprint Capacitor_SMD:C_0805_2012Metric_Pad1.18x1.45mm_HandSolder -> Capacitor_SMD:C_1206_3216Metric_Pad1.33x1.80mm_HandSolder
- C8: renamed from C6; value 2n -> 100n; footprint Capacitor_SMD:C_0805_2012Metric_Pad1.18x1.45mm_HandSolder -> Capacitor_SMD:C_1206_3216Metric_Pad1.33x1.80mm_HandSolder
- C9: renamed from C7; value 10n -> 100n; footprint Capacitor_SMD:C_0805_2012Metric_Pad1.18x1.45mm_HandSolder -> Capacitor_SMD:C_1206_3216Metric_Pad1.33x1.80mm_HandSolder
- CR1: renamed from CR2; footprint TVS:ZDO_TPSMF4L5.0A_LTF -> TVS:ZDO_TPSMF4L5.0A_LTF-L
- CR2: renamed from CR1; footprint TVS:ZDO_TPSMF4L5.0A_LTF -> TVS:ZDO_TPSMF4L5.0A_LTF-L
- CR3: footprint TVS:ZDO_TPSMF4L5.0A_LTF -> TVS:ZDO_TPSMF4L5.0A_LTF-L; moved to B.Cu
- R1: renamed from R17; value 1k -> 220
- R11: renamed from R8; footprint Package_SO:SO-16_3.9x9.9mm_P1.27mm -> Package_SO:SOIC-16_3.9x9.9mm_P1.27mm
- R15: renamed from R16; value 470 -> 100
- R21: renamed from R14; value 1k -> 100
- R3: renamed from R2; value 2k7 -> 2k7/910; footprint Resistor_SMD:R_0805_2012Metric_Pad1.20x1.40mm_HandSolder -> Resistor_SMD:R_1206_3216Metric_Pad1.30x1.75mm_HandSolder
- R7: renamed from R4; value 1k -> 100
- TH1: footprint Connector_PinHeader_1.27mm:PinHeader_2x02_P1.27mm_Vertical -> Connector_PinHeader_1.27mm:PinHeader_1x02_P1.27mm_Vertical
- moved J3 95.1 mm to (21.5, 33.8), turned to 180 degrees
- moved C28 79.2 mm to (68.5, 66.5)
- moved C7 78.9 mm to (64.5, 30.5), turned to 180 degrees
- moved C19 68.8 mm to (78.5, 66.5), turned to 180 degrees
- moved C17 64.2 mm to (85.0, 67.5)
- moved R18 63.3 mm to (94.5, 23.5)
- moved J10 61.9 mm to (111.5, 22.0)
- moved R22 59.3 mm to (97.5, 56.5)
- moved R23 58.5 mm to (97.5, 59.0)
- moved R12 56.2 mm to (63.0, 36.5)
- moved R1 48.1 mm to (113.5, 62.5)
- moved CR3 47.9 mm to (117.0, 47.5)
- moved R8 47.4 mm to (111.0, 71.0)
- moved C24 47.4 mm to (54.0, 67.0)
- moved U1 46.0 mm to (102.0, 67.5)
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- renumbered C15 to C12, C19 to C14, C31 to C18, C30 to C21, C27 to C22, C28 to C23, C29 to C24, C23 to C26, C33 to C29, D3 to D1, D4 to D2, D1 to D3, D2 to D4, J3 to J1, J7 to J10, J1 to J2, J2 to J3, J8 to J6, J9 to J7, J5 to J8, J6 to J9, R7 to R10, R18 to R12, R15 to R14, R20 to R16, R21 to R17, R26 to R18, R22 to R19, R1 to R2, R19 to R20, R25 to R22, R27 to R23, R23 to R24, R28 to R4, R3 to R5, R29 to R8, R5 to R9, U3 to U1, U1 to U3, U8 to U5, U5 to U6, U6 to U7
Connections:
- C10 pad 2: Net-(U1B-+) -> Net-(C10-Pad2)
- C11 pad 1: Net-(U1B-+) -> Net-(C10-Pad2)
- C14 pad 2: /7V_force -> Net-(C14-Pad2)
- C21 pad 2: Net-(U3C-V+) -> GND
- C28 pad 1: Net-(U3C-V+) -> Net-(U1C-V+)
- C3 pad 2: Net-(U1A-+) -> Net-(C3-Pad2)
- C4 pad 1: Net-(U1A-+) -> Net-(C3-Pad2)
- C5 pad 1: Net-(J1-Pin_2) -> Net-(J2-Pin_2)
- C6 pad 1: +15V -> +24V
- C8 pad 1: Net-(J1-Pin_2) -> Net-(J2-Pin_2)
- C9 pad 2: Net-(U1A--) (its old number) -> Net-(U3A--)
- CR2 pad 1: Net-(J1-Pin_2) -> Net-(J2-Pin_2)
- J2 pad 2: Net-(J1-Pin_2) -> Net-(J2-Pin_2)
- J3 pad 1: Net-(J2-Pin_1) -> Net-(J3-Pin_1)
- J3 pad 2: Net-(J2-Pin_2) -> Net-(J3-Pin_2)
- R10 pad 1: Net-(J1-Pin_2) -> Net-(J2-Pin_2)
- R11 pad 1: unconnected-(R8-Pad1) -> Net-(U3A--)
- R11 pad 10: Net-(R8-Pad10) -> Net-(JP2-A)
- R11 pad 11: Net-(R8-Pad10) -> Net-(JP2-A)
- R11 pad 12: Net-(R8-Pad12) -> Net-(JP2-A)
- R11 pad 13: Net-(J1-Pin_2) -> Net-(JP2-A)
- R11 pad 14: Net-(R8-Pad12) -> Net-(J2-Pin_2)
- R11 pad 15: Net-(R8-Pad10) -> Net-(J2-Pin_2)
- R11 pad 16: unconnected-(R8-Pad16) -> Net-(JP1-A)
- R11 pad 2: Net-(U1A--) (its old number) -> Net-(U3A--)
- R11 pad 3: GNDZ -> Net-(U3A--)
- R11 pad 4: Net-(U1A--) (its old number) -> Net-(U3A--)
- R11 pad 5: Net-(U1A--) (its old number) -> Net-(U3A--)
- R11 pad 6: Net-(U1A--) (its old number) -> GNDZ
- R11 pad 7: Net-(U1A--) (its old number) -> GNDZ
- R11 pad 8: unconnected-(R8-Pad8) -> GNDZ
- R11 pad 9: unconnected-(R8-Pad9) -> Net-(JP2-B)
- R12 pad 2: Net-(U1B-+) -> Net-(C10-Pad2)
- R15 pad 1: Net-(R16-Pad1) -> Net-(C14-Pad2)
- R16 pad 2: /7V_force -> Net-(C14-Pad2)
- R19 pad 2: /7V_force -> Net-(C14-Pad2)
- R3 pad 2: Net-(U2A--) -> Net-(Q1-E)
- R5 pad 2: Net-(U1A-+) -> Net-(C3-Pad2)
- R7 pad 2: Net-(J1-Pin_2) -> Net-(J2-Pin_2)
- TH1 pad 1: Net-(J2-Pin_2) -> Net-(J3-Pin_2)
- TH1 pad 2: Net-(J2-Pin_2) -> Net-(J3-Pin_1)
- TP2 pad 1: /7V_force -> Net-(C14-Pad2)
- U1 pad 8: Net-(U3C-V+) -> Net-(U1C-V+)
- U2 pad 1: Net-(U2A--) -> Net-(Q1-B)
- U2 pad 2: Net-(U2A--) -> Net-(Q1-E)
- U2 pad 3: Net-(J1-Pin_2) -> Net-(J2-Pin_2)
- U2 pad 7: Net-(R16-Pad1) -> Net-(C14-Pad2)
- U3 pad 2: Net-(U1A--) (its old number) -> Net-(U3A--)
- U3 pad 3: Net-(U1A-+) -> Net-(U3A-+)
- U3 pad 5: Net-(U1B-+) -> Net-(U3B-+)
- U4 pad 3: +15V -> +24V
- U7 pad 3: Net-(U3C-V+) -> Net-(U1C-V+)
Routing:
- net +15V: track 0.00 -> 116.1 mm, vias 0 -> 3
- net Net-(J2-Pin_2): track 0.00 -> 73.6 mm, vias 0 -> 2
- net Net-(U1C-V+): track 0.00 -> 51.0 mm, vias 0 -> 1
- net Net-(D3-K): track 0.00 -> 47.5 mm
- net GNDZ: track 0.00 -> 35.7 mm
- net Net-(C14-Pad2): track 0.00 -> 31.5 mm
- net /GND1F: track 0.00 -> 28.5 mm
- net /GND1S: track 0.00 -> 27.6 mm
- net Net-(C3-Pad2): track 0.00 -> 24.2 mm
- net Net-(C16-Pad2): track 0.00 -> 24.2 mm, vias 0 -> 2
- net Net-(D1-A): track 0.00 -> 21.7 mm
- net /7V_force: track 0.00 -> 20.8 mm
- net Net-(C10-Pad2): track 0.00 -> 18.0 mm
- net Net-(U3A--): track 0.00 -> 17.7 mm
- net /GND2S: track 0.00 -> 16.8 mm
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Other:
- board size 108 x 55.5 mm -> 107.5 x 55.5 mm

Commit message: Update KiCad project and add latest backups
Parts:
- removed TP1: GNDZ, TestPoint:TestPoint_Pad_1.5x1.5mm
- removed TP2: ~, TestPoint:TestPoint_Pad_1.5x1.5mm
- added C20: 100n, Capacitor_SMD:C_0805_2012Metric_Pad1.18x1.45mm_HandSolder, F.Cu at (106.0, 43.5)
- added J11: Conn_01x01, Connector_Wire:SolderWire-1sqmm_1x01_D1.4mm_OD3.9mm, F.Cu at (61.0, 26.5)
- added NT3: NetTie_3, Jumper:SolderJumper-3_P2.0mm_Open_TrianglePad1.0x1.5mm_NumberLabels, F.Cu at (31.0, 37.5)
- added R25: 220k, Resistor_SMD:R_0805_2012Metric_Pad1.20x1.40mm_HandSolder, F.Cu at (113.5, 41.0)
- added R26: 51, Resistor_SMD:R_0805_2012Metric_Pad1.20x1.40mm_HandSolder, F.Cu at (116.0, 39.0)
- added R27: 51k, Resistor_SMD:R_0805_2012Metric_Pad1.20x1.40mm_HandSolder, F.Cu at (101.5, 39.0)
- added R28: 51, Resistor_SMD:R_0805_2012Metric_Pad1.20x1.40mm_HandSolder, F.Cu at (99.0, 39.0)
- added U8: OPA2182xD, Package_SO:SOIC-8_3.9x4.9mm_P1.27mm, F.Cu at (107.5, 39.0)
- C6: moved to F.Cu
- C7: value 10n -> 330n
- NT2: moved to B.Cu
- R9: footprint Resistor_SMD:R_0805_2012Metric_Pad1.20x1.40mm_HandSolder -> Resistor_SMD:R_1206_3216Metric_Pad1.30x1.75mm_HandSolder
- moved NT2 13.6 mm to (36.5, 51.0)
- moved C8 8.42 mm to (117.4, 31.6)
- moved CR2 8.42 mm to (120.9, 31.6)
- moved J2 8.42 mm to (125.4, 30.3)
- moved R10 8.41 mm to (113.5, 31.6)
- moved J4 7.07 mm to (123.2, 37.2)
- moved C6 4.00 mm to (34.5, 32.5)
- moved NT1 3.20 mm to (62.5, 25.5), turned to -160 degrees
- moved TH1 2.55 mm to (28.0, 31.0)
- moved R9 0.50 mm to (64.5, 33.0)
Connections:
- net Net-(D1-A) renamed -12V
- net Net-(R12-Pad1) renamed /Vz
- C6 pad 2: GND -> Net-(C6-Pad2)
- J4 pad 1: GND -> /G1F100
- J4 pad 3: GNDZ -> /GND400
- J4 pad 4: GNDZ -> GND
- U4 pad 4: GND -> Net-(C6-Pad2)
Routing:
- net Net-(U1C-V-): track 16.7 -> 83.5 mm, vias 0 -> 2
- net -12V: track 21.7 -> 84.1 mm
- net /7V_sense: track 0.00 -> 49.8 mm, vias 0 -> 1
- net /Vz: track 3.02 -> 39.4 mm
- net +15V: track 116.1 -> 149.7 mm
- net +24V: track 0.00 -> 32.9 mm, vias 0 -> 1
- net /G1F100: track 0.00 -> 30.5 mm, vias 0 -> 1
- net /GND1F: track 28.5 -> 55.2 mm, vias 0 -> 2
- net Net-(C14-Pad2): track 31.5 -> 57.4 mm
- net Net-(U1C-V+): track 51.0 -> 74.4 mm, vias 1 -> 2
- net GNDZ: track 35.7 -> 57.5 mm
- net Net-(C6-Pad2): track 0.00 -> 21.7 mm
- net /GND400: track 0.00 -> 15.4 mm
- net Net-(J2-Pin_2): track 73.6 -> 87.3 mm, vias 2 -> 3
- net Net-(J3-Pin_1): track 0.00 -> 7.12 mm
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
Commit message: Update KiCad project and backup files- just before format R9 7900x SSD
Parts:
- added C31: 100n, Capacitor_SMD:C_0805_2012Metric_Pad1.18x1.45mm_HandSolder, B.Cu at (67.5, 60.0)
- moved R14 37.3 mm to (85.5, 62.0), turned to 0 degrees
- moved Q1 0.50 mm to (73.5, 54.5)
Routing:
- net Net-(C13-Pad2): track 6.44 -> 55.2 mm, vias 0 -> 2
- net Net-(C10-Pad2): track 18.0 -> 25.0 mm
- net Net-(U2B-+): track 2.12 -> 4.64 mm
- net +15V: track 149.7 -> 150.6 mm
- net Net-(Q1-E): track 15.4 -> 16.2 mm
- net Net-(Q1-B): track 10.4 -> 9.85 mm
