File: ADR1399New/ADR1399.kicad_sch (KiCad schematic)
At the start: 78 parts, among them J1 10V, J2 PT100, J3 GNDF_SPARE, J4 7V, J5 Conn_01x02_Male, J6 Conn_01x02_Male, J7 Conn_01x01_Male, J8 Conn_01x02_Male, J9 Conn_01x02_Male, U1 OPA2182xD, U2 OPA2209xD, U3 OPA2182xD, U4 LM399, U5 LM7815_TO220, U6 LM7805_TO220, U8 LM7905_TO220

Commit message: Update KiCad project and add latest backups
Parts:
- removed C26: 100n, Capacitor_SMD:C_0805_2012Metric_Pad1.18x1.45mm_HandSolder, symbol Device:C
- removed C8: 2n2, Capacitor_SMD:C_0805_2012Metric_Pad1.18x1.45mm_HandSolder, symbol Device:C
- removed TH1: PT1000, Connector_PinHeader_1.27mm:PinHeader_2x02_P1.27mm_Vertical, symbol Device:Thermistor_PTC_4Wire
- added C30: 100n, Capacitor_SMD:C_0805_2012Metric_Pad1.18x1.45mm_HandSolder, symbol Device:C
- added H1, H2, H3, H4: 3mm, MountingHole:MountingHole_3.2mm_M3, symbol Mechanical:MountingHole
- added J4: Guards, Connector_PinHeader_2.54mm:PinHeader_2x02_P2.54mm_Vertical, symbol Connector:Conn_01x04_Pin
- added JP1: 3k3/5k, Jumper:SolderJumper-2_P1.3mm_Bridged2Bar_RoundedPad1.0x1.5mm, symbol Jumper:Jumper_2_Small_Bridged
- added JP2: 8k33/10k, Jumper:SolderJumper-2_P1.3mm_Bridged2Bar_RoundedPad1.0x1.5mm, symbol Jumper:Jumper_2_Small_Bridged
- added NT2: NetTie_2, NetTie:NetTie-2_SMD_Pad2.0mm, symbol Device:NetTie_2
- added Q1: BC817, Package_TO_SOT_SMD:SOT-23, symbol Transistor_BJT:BC817
- added R13, R6: 33, Resistor_SMD:R_0805_2012Metric_Pad1.20x1.40mm_HandSolder, symbol Device:R
- added TH1: PT1000, Connector_PinHeader_1.27mm:PinHeader_1x02_P1.27mm_Vertical, symbol Sensor_Temperature:PT1000
- added TP1: GNDZ, TestPoint:TestPoint_Pad_1.5x1.5mm, symbol Connector:TestPoint
- C1: renamed from C14; value 2n -> 100n; footprint Capacitor_SMD:C_0805_2012Metric_Pad1.18x1.45mm_HandSolder -> Capacitor_SMD:C_1206_3216Metric_Pad1.33x1.80mm_HandSolder
- C10: renamed from C17; footprint Capacitor_THT:C_Rect_L7.2mm_W4.5mm_P5.00mm_FKS2_FKP2_MKS2_MKP2 -> Capacitor_THT:C_Rect_L7.2mm_W5.5mm_P5.00mm_FKS2_FKP2_MKS2_MKP2
- C11: renamed from C18; value 10n -> 1n
- C13: renamed from C20; value 22n -> 100n; footprint Capacitor_SMD:C_0805_2012Metric_Pad1.18x1.45mm_HandSolder -> Capacitor_SMD:C_1206_3216Metric_Pad1.33x1.80mm_HandSolder
- C15: renamed from C16; value 2n -> 100p; footprint Capacitor_SMD:C_0805_2012Metric_Pad1.18x1.45mm_HandSolder -> Capacitor_SMD:C_1206_3216Metric_Pad1.33x1.80mm_HandSolder
- C16: renamed from C34; footprint Capacitor_SMD:C_0805_2012Metric_Pad1.18x1.45mm_HandSolder -> Capacitor_SMD:C_1206_3216Metric_Pad1.33x1.80mm_HandSolder
- C17: renamed from C22; value C -> 100n; footprint Capacitor_SMD:C_1206_3216Metric -> Capacitor_SMD:C_1206_3216Metric_Pad1.33x1.80mm_HandSolder
- C19: renamed from C32; footprint Capacitor_SMD:C_1206_3216Metric -> Capacitor_Tantalum_SMD:CP_EIA-3528-12_Kemet-T_HandSolder
- C2: renamed from C35; footprint Capacitor_SMD:C_0805_2012Metric_Pad1.18x1.45mm_HandSolder -> Capacitor_SMD:C_1206_3216Metric_Pad1.33x1.80mm_HandSolder
- C25: renamed from C21; value C -> 100n; footprint Capacitor_SMD:C_1206_3216Metric -> Capacitor_SMD:C_1206_3216Metric_Pad1.33x1.80mm_HandSolder
- C27: renamed from C24; value 100.0 -> 220.0; footprint Capacitor_SMD:C_1206_3216Metric -> Capacitor_THT:CP_Radial_D10.0mm_P7.50mm
- C28: renamed from C25; footprint Capacitor_SMD:C_1206_3216Metric -> Capacitor_Tantalum_SMD:CP_EIA-3528-12_Kemet-T_HandSolder
- C3: renamed from C1; footprint Capacitor_THT:C_Rect_L7.2mm_W4.5mm_P5.00mm_FKS2_FKP2_MKS2_MKP2 -> Capacitor_THT:C_Rect_L7.2mm_W5.5mm_P5.00mm_FKS2_FKP2_MKS2_MKP2
- C4: renamed from C2; value 10n -> 1n
- C5: renamed from C3; footprint Capacitor_SMD:C_0805_2012Metric_Pad1.18x1.45mm_HandSolder -> Capacitor_SMD:C_1206_3216Metric_Pad1.33x1.80mm_HandSolder
- C6: renamed from C4; footprint Capacitor_SMD:C_0805_2012Metric_Pad1.18x1.45mm_HandSolder -> Capacitor_SMD:C_1206_3216Metric_Pad1.33x1.80mm_HandSolder
- C7: renamed from C5; footprint Capacitor_SMD:C_0805_2012Metric_Pad1.18x1.45mm_HandSolder -> Capacitor_SMD:C_1206_3216Metric_Pad1.33x1.80mm_HandSolder
- C8: renamed from C6; value 2n -> 100n; footprint Capacitor_SMD:C_0805_2012Metric_Pad1.18x1.45mm_HandSolder -> Capacitor_SMD:C_1206_3216Metric_Pad1.33x1.80mm_HandSolder
- C9: renamed from C7; value 10n -> 100n; footprint Capacitor_SMD:C_0805_2012Metric_Pad1.18x1.45mm_HandSolder -> Capacitor_SMD:C_1206_3216Metric_Pad1.33x1.80mm_HandSolder
- CR1: renamed from CR2; footprint TVS:ZDO_TPSMF4L5.0A_LTF -> TVS:ZDO_TPSMF4L5.0A_LTF-L
- CR2: renamed from CR1; footprint TVS:ZDO_TPSMF4L5.0A_LTF -> TVS:ZDO_TPSMF4L5.0A_LTF-L
- CR3: footprint TVS:ZDO_TPSMF4L5.0A_LTF -> TVS:ZDO_TPSMF4L5.0A_LTF-L
- J5: renamed from J4; footprint (none) -> Connector_PinHeader_2.54mm:PinHeader_1x04_P2.54mm_Vertical
- NT1: footprint (none) -> NetTie:NetTie-2_SMD_Pad2.0mm
- R1: renamed from R17; value 1k -> 220
- R11: renamed from R8; footprint Package_SO:SO-16_3.9x9.9mm_P1.27mm -> Package_SO:SOIC-16_3.9x9.9mm_P1.27mm
- R15: renamed from R16; value 470 -> 100
- R21: renamed from R14; value 1k -> 100
- R3: renamed from R2; value 2k7 -> 2k7/910; footprint Resistor_SMD:R_0805_2012Metric_Pad1.20x1.40mm_HandSolder -> Resistor_SMD:R_1206_3216Metric_Pad1.30x1.75mm_HandSolder
- R7: renamed from R4; value 1k -> 100
- renumbered C15 to C12, C19 to C14, C31 to C18, C30 to C21, C27 to C22, C28 to C23, C29 to C24, C23 to C26, C33 to C29, D3 to D1, D4 to D2, D1 to D3, D2 to D4, J3 to J1, J7 to J10, J1 to J2, J2 to J3, J8 to J6, J9 to J7, J5 to J8, J6 to J9, R7 to R10, R18 to R12, R15 to R14, R20 to R16, R21 to R17, R26 to R18, R22 to R19, R1 to R2, R19 to R20, R25 to R22, R27 to R23, R23 to R24, R28 to R4, R3 to R5, R29 to R8, R5 to R9, U3 to U1, U1 to U3, U8 to U5, U5 to U6, U6 to U7
Connections:
- net +15V: now also NT2.1, Q1.3 (C); no longer C6.1, U4.3
- net 7V_force: no longer C14.2, R16.2, R19.2, TP2.1
- net GND: now also C21.2, C30.1, J4.1 (Pin_1), J4.2 (Pin_2)
- net GNDZ: now also R11.6, R11.7, R11.8, J4.3 (Pin_3), J4.4 (Pin_4), TP1.1; no longer R11.3
- net at R11.1: now also C9.2, R11.2, R11.3, R11.4, R11.5, U3.2 (-)
- net at R11.10, R11.11: now also R11.12, R11.13, JP2.1 (A); no longer R11.15
- net at R11.14: now also C5.1, C8.1, CR2.1, J2.2 (Pin_2), R10.1, R11.15, R7.2, U2.3 (+), JP1.2 (B); no longer R11.12
- net at R11.16: now also JP1.1 (A)
- net at R11.9: now also JP2.2 (B)
- net at C28.1, U1.8 (V+), U7.3 (VO): now also C30.2; no longer C21.2
- net at R3.2, U2.2 (-): now also Q1.2 (E); no longer U2.1
- net at C3.2, C4.1, R5.2: now also R6.1; no longer U3.3 (+)
- net at R15.1, U2.7: now also C14.2, R16.2, R19.2, TP2.1
- net at J3.1 (Pin_1): now also TH1.2
- net at J3.2 (Pin_2): now also TH1.1
- net at C10.2, C11.1, R12.2: now also R13.1; no longer U3.5 (+)
- new net: Q1.1 (B), U2.1
- new net: R13.2, U3.5 (+)
- new net: R6.2, U3.3 (+)
- new net +24V: C6.1, NT2.2, U4.3
- no-connect marks 4 -> 0
Other:
- moved on the sheet: C10, C11, C21, C3, C4, C7, CR3, R11, R12, R15, R3, R5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

Commit message: Update KiCad project and add latest backups
Parts:
- removed TP1: GNDZ, TestPoint:TestPoint_Pad_1.5x1.5mm, symbol Connector:TestPoint
- removed TP2: ~, TestPoint:TestPoint_Pad_1.5x1.5mm, symbol Connector:TestPoint
- added C20: 100n, Capacitor_SMD:C_0805_2012Metric_Pad1.18x1.45mm_HandSolder, symbol Device:C
- added J11: Conn_01x01, Connector_Wire:SolderWire-1sqmm_1x01_D1.4mm_OD3.9mm, symbol Connector_Generic:Conn_01x01
- added NT3: NetTie_3, Jumper:SolderJumper-3_P2.0mm_Open_TrianglePad1.0x1.5mm_NumberLabels, symbol Device:NetTie_3
- added R25: 220k, Resistor_SMD:R_0805_2012Metric_Pad1.20x1.40mm_HandSolder, symbol Device:R
- added R26, R28: 51, Resistor_SMD:R_0805_2012Metric_Pad1.20x1.40mm_HandSolder, symbol Device:R
- added R27: 51k, Resistor_SMD:R_0805_2012Metric_Pad1.20x1.40mm_HandSolder, symbol Device:R
- added U8: OPA2182xD, Package_SO:SOIC-8_3.9x4.9mm_P1.27mm, symbol Amplifier_Operational:OPA2196xD
- C7: value 10n -> 330n
- R9: footprint Resistor_SMD:R_0805_2012Metric_Pad1.20x1.40mm_HandSolder -> Resistor_SMD:R_1206_3216Metric_Pad1.30x1.75mm_HandSolder
Connections:
- net GND: now also J4.4 (Pin_4), NT3.1, R26.2, R28.2; no longer C6.2, J4.1 (Pin_1), U4.4
- net GND1F: now also U8.5 (+)
- net GNDZ: now also J11.1 (Pin_1), U8.3 (+); no longer J4.3 (Pin_3), J4.4 (Pin_4)
- net -12V: now reaches C17.1, C18.1, D1.2 (A), D2.2 (A), U5.2 (VI)
- net -12V: now also NT3.3
- net at C19.1, C21.1, U1.4 (V-)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: now also C20.1, U8.4 (V-)
- net at C28.1, C30.2, U1.8 (V+)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: now also C20.2, U8.8 (V+)
- net Vz: now reaches R12.1, R2.2, R3.1, R5.1, R9.1, U4.1
- new net: R27.1, R28.1, U8.6 (-)
- new net: C6.2, NT3.2, U4.4
- new net: R25.1, R26.1, U8.2 (-)
- new net G1F100: J4.1 (Pin_1), R27.2, U8.7
- new net GND400: J4.3 (Pin_3), R25.2, U8.1
Other:
- moved on the sheet: C21, C30, C6, J4

Commit message: Update KiCad project and backup files- just before format R9 7900x SSD
Parts:
- added C31: 100n, Capacitor_SMD:C_0805_2012Metric_Pad1.18x1.45mm_HandSolder, symbol Device:C
Connections:
- net +15V: now also C31.1
- net GND: now also C31.2
Other:
- moved on the sheet: C24, NT2
Changed lines of the file:
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@@
 	)
 	(junction
+		(at 134.62 163.83)
+		(diameter 0)
+		(color 0 0 0 0)
+	)
+	(junction
 		(at 31.75 63.5)
 		(diameter 0)
@@
 	)
 	(junction
+		(at 142.24 163.83)
+		(diameter 0)
+		(color 0 0 0 0)
+	)
+	(junction
 		(at 129.54 57.15)
 		(diameter 0)
@@
 	)
 	(junction
-		(at 135.89 163.83)
-		(diameter 0)
-		(color 0 0 0 0)
-	)
-	(junction
 		(at 63.5 180.34)
 		(diameter 0)
@@
 	)
 	(junction
+		(at 134.62 180.34)
+		(diameter 0)
+		(color 0 0 0 0)
+	)
+	(junction
 		(at 63.5 154.94)
 		(diameter 0)
@@
 	(wire
 		(pts
-			(xy 147.32 162.56) (xy 147.32 163.83)
+			(xy 149.86 162.56) (xy 149.86 163.83)
 		)
 		(stroke
@@
 	(wire
 		(pts
-			(xy 127 180.34) (xy 135.89 180.34)
+			(xy 127 180.34) (xy 134.62 180.34)
 		)
 		(stroke
@@
 	(wire
 		(pts
+			(xy 134.62 180.34) (xy 142.24 180.34)
+		)
+		(stroke
+			(width 0)
+			(type default)
+		)
+	)
+	(wire
+		(pts
 			(xy 132.08 97.79) (xy 137.16 97.79)
 		)
@@
 	(wire
 		(pts
-			(xy 127 163.83) (xy 135.89 163.83)
+			(xy 127 163.83) (xy 134.62 163.83)
 		)
 		(stroke
@@
 	(wire
 		(pts
+			(xy 142.24 163.83) (xy 143.51 163.83)
+		)
+		(stroke
+			(width 0)
+			(type default)
+		)
+	)
+	(wire
+		(pts
 			(xy 68.58 57.15) (xy 68.58 58.42)
 		)
@@
 	(wire
 		(pts
-			(xy 135.89 163.83) (xy 139.7 163.83)
-		)
-		(stroke
-			(width 0)
-			(type default)
-		)
-	)
-	(wire
-		(pts
 			(xy 115.57 149.86) (xy 115.57 151.13)
 		)
@@
 	(wire
 		(pts
+			(xy 142.24 163.83) (xy 142.24 168.91)
+		)
+		(stroke
+			(width 0)
+			(type default)
+		)
+	)
+	(wire
+		(pts
 			(xy 123.19 105.41) (xy 123.19 110.49)
 		)
@@
 	(wire
 		(pts
-			(xy 135.89 176.53) (xy 135.89 180.34)
+			(xy 134.62 176.53) (xy 134.62 180.34)
 		)
 		(stroke
@@
 	(wire
 		(pts
-			(xy 144.78 163.83) (xy 147.32 163.83)
+			(xy 148.59 163.83) (xy 149.86 163.83)
 		)
 		(stroke
@@
 	(wire
 		(pts
-			(xy 135.89 163.83) (xy 135.89 168.91)
+			(xy 134.62 163.83) (xy 134.62 168.91)
 		)
 		(stroke
@@
 	(wire
 		(pts
+			(xy 142.24 176.53) (xy 142.24 180.34)
+		)
+		(stroke
+			(width 0)
+			(type default)
+		)
+	)
+	(wire
+		(pts
 			(xy 185.42 34.29) (xy 189.23 34.29)
 		)
@@
 	(wire
 		(pts
+			(xy 134.62 163.83) (xy 142.24 163.83)
+		)
+		(stroke
+			(width 0)
+			(type default)
+		)
+	)
+	(wire
+		(pts
 			(xy 127 78.74) (xy 127 80.01)
 		)
@@
 	(symbol
 		(lib_id "Device:NetTie_2")
-		(at 142.24 163.83 0)
+		(at 146.05 163.83 0)
 		(unit 1)
 		(exclude_from_sim no)
@@
 		(dnp no)
 		(property "Reference" "NT2"
-			(at 141.986 160.782 0)
+			(at 145.796 161.798 0)
 			(effects
 				(font
@@
 		)
 		(property "Value" "NetTie_2"
-			(at 142.24 161.29 0)
+			(at 146.05 161.29 0)
 			(effects
 				(font
@@
 		)
 		(property "Footprint" "NetTie:NetTie-2_SMD_Pad2.0mm"
-			(at 142.24 163.83 0)
+			(at 146.05 163.83 0)
 			(effects
 				(font
@@
 		)
 		(property "Datasheet" "~"
-			(at 142.24 163.83 0)
+			(at 146.05 163.83 0)
 			(effects
 				(font
@@
 		)
 		(property "Description" "Net tie, 2 pins"
-			(at 142.24 163.83 0)
+			(at 146.05 163.83 0)
 			(effects
 				(font
@@
 	(symbol
 		(lib_id "power:+24V")
-		(at 147.32 162.56 0)
+		(at 149.86 162.56 0)
 		(unit 1)
 		(exclude_from_sim no)
@@
 		(fields_autoplaced yes)
 		(property "Reference" "#PWR022"
-			(at 147.32 166.37 0)
+			(at 149.86 166.37 0)
 			(effects
 				(font
@@
 		)
 		(property "Value" "+24V"
-			(at 147.32 157.48 0)
+			(at 149.86 157.48 0)
 			(effects
 				(font
@@
 		)
 		(property "Footprint" ""
-			(at 147.32 162.56 0)
+			(at 149.86 162.56 0)
 			(effects
 				(font
@@
 		)
 		(property "Datasheet" ""
-			(at 147.32 162.56 0)
+			(at 149.86 162.56 0)
 			(effects
 				(font
@@
 		)
 		(property "Description" "Power symbol creates a global label with name \"+24V\""
-			(at 147.32 162.56 0)
+			(at 149.86 162.56 0)
 			(effects
 				(font
@@
 	)
 	(symbol
+		(lib_id "Device:C")
+		(at 142.24 172.72 0)
+		(unit 1)
+		(exclude_from_sim no)
+		(in_bom yes)
+		(on_board yes)
+		(dnp no)
+		(property "Reference" "C31"
+			(at 143.51 170.18 0)
+			(effects
+				(font
+					(size 1.27 1.27)
+				)
+				(justify left)
+			)
+		)
+		(property "Value" "100n"
+			(at 143.51 175.26 0)
+			(effects
+				(font
+					(size 1.27 1.27)
+				)
+				(justify left)
+			)
+		)
+		(property "Footprint" "Capacitor_SMD:C_0805_2012Metric_Pad1.18x1.45mm_HandSolder"
+			(at 143.2052 176.53 0)
+			(effects
+				(font
+					(size 1.27 1.27)
+				)
+				(hide yes)
+			)
+		)
+		(property "Datasheet" "~"
+			(at 142.24 172.72 0)
+			(effects
+				(font
+					(size 1.27 1.27)
+				)
+				(hide yes)
+			)
+		)
+		(property "Description" "Unpolarized capacitor"
+			(at 142.24 172.72 0)
+			(effects
+				(font
+					(size 1.27 1.27)
+				)
+				(hide yes)
+			)
+		)
+		(pin "1"
+		)
+		(pin "2"
+		)
+		(instances
+			(project "ADR1399"
+				(path "/e63e39d7-6ac0-4ffd-8aa3-1841a4541b55"
+					(reference "C31")
+					(unit 1)
+				)
+			)
+		)
+	)
+	(symbol
 		(lib_id "Device:R")
 		(at 39.37 187.96 0)
@@
 		(dnp no)
 		(property "Reference" "C23"
-			(at 128.27 170.18 0)
+			(at 128.016 170.18 0)
 			(effects
 				(font
@@
 	(symbol
 		(lib_id "Device:C")
-		(at 135.89 172.72 0)
+		(at 134.62 172.72 0)
 		(unit 1)
 		(exclude_from_sim no)
@@
 		(dnp no)
 		(property "Reference" "C24"
-			(at 137.16 170.18 0)
+			(at 135.89 170.18 0)
 			(effects
 				(font
@@
 		)
 		(property "Value" "100n"
-			(at 137.16 175.26 0)
+			(at 135.89 175.26 0)
 			(effects
 				(font
@@
 		)
 		(property "Footprint" "Capacitor_SMD:C_0805_2012Metric_Pad1.18x1.45mm_HandSolder"
-			(at 136.8552 176.53 0)
+			(at 135.5852 176.53 0)
 			(effects
 				(font
@@
 		)
 		(property "Datasheet" "~"
-			(at 135.89 172.72 0)
+			(at 134.62 172.72 0)
 			(effects
 				(font
@@
 		)
 		(property "Description" "Unpolarized capacitor"
-			(at 135.89 172.72 0)
+			(at 134.62 172.72 0)
 			(effects
 				(font
